File: pcb/display_unit/display_unit.kicad_pcb (KiCad board)
At the start: 2 copper layers, 80 x 40 mm, 20 parts, among them J3 Conn_01x05, J4 Conn_01x06, M1 ROTARY-ENCODER, M2 096_INCH_OLED, Q1 Q_NMOS_GDS, T1 TERMINAL_ELEMENT14_5MM_X3, T2 TERMINAL_ELEMENT14_5MM_X2, T3 TERMINAL_ELEMENT14_5MM_X2, T4 TERMINAL_ELEMENT14_5MM_X2, U1 LM2936-3.3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

Commit message: Added pull down resistor on led light driver
Parts:
- added R2: R, Resistors_SMD:R_0805_HandSoldering, F.Cu at (107.4, 96.8)
Routing:
- net /LIGHT: track 72.2 -> 75.6 mm, vias 1 -> 2
Changed lines of the file:
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@@
 (kicad_pcb (version 4) (host pcbnew 4.0.7-e2-6376~58~ubuntu16.04.1)
   (general
-    (links 55)
+    (links 57)
     (no_connects 0)
     (area 77.924999 61.924999 158.075001 102.075001)
     (thickness 1.6)
     (drawings 31)
-    (tracks 195)
+    (tracks 199)
     (zones 0)
-    (modules 20)
+    (modules 21)
     (nets 22)
   )
@@
       (net 1 VDD))
   )
+  (module Resistors_SMD:R_0805_HandSoldering (layer F.Cu)
+    (at 107.4 96.75)
+    (descr "Resistor SMD 0805, hand soldering")
+    (tags "resistor 0805")
+    (attr smd)
+    (fp_text reference R2 (at 0 -1.7) (layer F.SilkS)
+      (effects (font (size 1 1) (thickness 0.15)))
+    )
+    (fp_text value R (at 0 1.75) (layer F.Fab)
+      (effects (font (size 1 1) (thickness 0.15)))
+    )
+    (fp_text user %R (at 0 0) (layer F.Fab)
+      (effects (font (size 0.5 0.5) (thickness 0.075)))
+    )
+    (fp_line (start -1 0.62) (end -1 -0.62) (layer F.Fab) (width 0.1))
+    (fp_line (start 1 0.62) (end -1 0.62) (layer F.Fab) (width 0.1))
+    (fp_line (start 1 -0.62) (end 1 0.62) (layer F.Fab) (width 0.1))
+    (fp_line (start -1 -0.62) (end 1 -0.62) (layer F.Fab) (width 0.1))
+    (fp_line (start 0.6 0.88) (end -0.6 0.88) (layer F.SilkS) (width 0.12))
+    (fp_line (start -0.6 -0.88) (end 0.6 -0.88) (layer F.SilkS) (width 0.12))
+    (fp_line (start -2.35 -0.9) (end 2.35 -0.9) (layer F.CrtYd) (width 0.05))
+    (fp_line (start -2.35 -0.9) (end -2.35 0.9) (layer F.CrtYd) (width 0.05))
+    (fp_line (start 2.35 0.9) (end 2.35 -0.9) (layer F.CrtYd) (width 0.05))
+    (fp_line (start 2.35 0.9) (end -2.35 0.9) (layer F.CrtYd) (width 0.05))
+    (pad 1 smd rect (at -1.35 0) (size 1.5 1.3) (layers F.Cu F.Paste F.Mask)
+      (net 17 /LIGHT))
+    (pad 2 smd rect (at 1.35 0) (size 1.5 1.3) (layers F.Cu F.Paste F.Mask)
+      (net 2 GND))
+    (model ${KISYS3DMOD}/Resistors_SMD.3dshapes/R_0805.wrl
+      (at (xyz 0 0 0))
+      (scale (xyz 1 1 1))
+      (rotate (xyz 0 0 0))
+    )
+  )
   (gr_line (start 78 62) (end 158 62) (angle 90) (layer Edge.Cuts) (width 0.15))
   (gr_line (start 78 102) (end 158 102) (angle 90) (layer Edge.Cuts) (width 0.15))
@@
     (effects (font (size 1.5 1.5) (thickness 0.3)))
   )
-  (gr_text +3V3 (at 150.5 78 360) (layer F.SilkS)
-    (effects (font (size 1.5 1.5) (thickness 0.3)))
-  )
-  (gr_text SWDIO (at 150.5 75.5 360) (layer F.SilkS)
-    (effects (font (size 1.5 1.5) (thickness 0.3)))
-  )
-  (gr_text SWCLK (at 150.5 73 360) (layer F.SilkS)
-    (effects (font (size 1.5 1.5) (thickness 0.3)))
-  )
-  (gr_text NRST (at 151 70.5 360) (layer F.SilkS)
-    (effects (font (size 1.5 1.5) (thickness 0.3)))
-  )
-  (gr_text "GND\n" (at 151.5 68 360) (layer F.SilkS)
+  (gr_text +3V3 (at 150.5 78) (layer F.SilkS)
+    (effects (font (size 1.5 1.5) (thickness 0.3)))
+  )
+  (gr_text SWDIO (at 150.5 75.5) (layer F.SilkS)
+    (effects (font (size 1.5 1.5) (thickness 0.3)))
+  )
+  (gr_text SWCLK (at 150.5 73) (layer F.SilkS)
+    (effects (font (size 1.5 1.5) (thickness 0.3)))
+  )
+  (gr_text NRST (at 151 70.5) (layer F.SilkS)
+    (effects (font (size 1.5 1.5) (thickness 0.3)))
+  )
+  (gr_text "GND\n" (at 151.5 68) (layer F.SilkS)
     (effects (font (size 1.5 1.5) (thickness 0.3)))
   )
@@
   (segment (start 136.62 77.202081) (end 134.13 79.692081) (width 0.6) (layer F.Cu) (net 16))
   (segment (start 134.13 79.692081) (end 134.13 89.838616) (width 0.6) (layer F.Cu) (net 16))
+  (segment (start 103.75 96.75) (end 106.05 96.75) (width 0.6) (layer F.Cu) (net 17))
+  (segment (start 104.5 96) (end 103.75 96.75) (width 0.6) (layer B.Cu) (net 17))
+  (via (at 103.75 96.75) (size 0.6) (drill 0.4) (layers F.Cu B.Cu) (net 17))
+  (segment (start 104.5 96) (end 89.5 81) (width 0.6) (layer B.Cu) (net 17))
+  (segment (start 108.30001 99.80001) (end 104.5 96) (width 0.6) (layer B.Cu) (net 17))
   (segment (start 145 98.1) (end 143.29999 99.80001) (width 0.6) (layer B.Cu) (net 17))
   (segment (start 143.29999 99.80001) (end 108.30001 99.80001) (width 0.6) (layer B.Cu) (net 17))
-  (segment (start 108.30001 99.80001) (end 89.5 81) (width 0.6) (layer B.Cu) (net 17))
   (segment (start 89.5 81) (end 88 81) (width 0.6) (layer B.Cu) (net 17))
   (segment (start 143.3 97.5) (end 143.9 98.1) (width 0.6) (layer F.Cu) (net 17))
