File: pcb/display_unit/display_unit.kicad_pcb (KiCad board)
At the start: 2 copper layers, 80 x 40 mm, 21 parts, among them J3 Conn_01x05, J4 Conn_01x06, M1 ROTARY-ENCODER, M2 096_INCH_OLED, Q1 Q_NMOS_GDS, T1 TERMINAL_ELEMENT14_5MM_X3, T2 TERMINAL_ELEMENT14_5MM_X2, T3 TERMINAL_ELEMENT14_5MM_X2, T4 TERMINAL_ELEMENT14_5MM_X2, U1 LM2936-3.3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

Commit message: Got oled working.
Parts:
- C1: value CP -> 10uf 25v
- C5: value CP -> 10uf 6.3v
- Q1: value Q_NMOS_GDS -> NVD6828NLT4G; footprint TO_SOT_Packages_THT:TO-220-3_Horizontal -> TO_SOT_Packages_SMD:TO-252-2
- R2: value R -> 100K
- U1: value LM2936-3.3 -> UA78M33CDCY
- U2: footprint Housings_QFP:LQFP-32_7x7mm_Pitch0.8mm -> custom_microcontroller:LQFP-32_7x7mm_Pitch0.8mm
- moved Q1 5.06 mm to (85.5, 85.4), turned to 270 degrees
Routing:
- net Net-(Q1-Pad2): track 7.60 -> 25.1 mm, vias 0 -> 1
- net /LIGHT: track 75.6 -> 75.9 mm, vias 2 -> 3
