File: pcb/relay_unit/relay_unit.kicad_pcb (KiCad board)
At the start: 2 copper layers, 105 x 55 mm, 29 parts, among them J3 Conn_01x05, J4 Conn_01x06, K1 TE_OJ_Series, K2 TE_OJ_Series, K3 TE_OJ_Series, Q1 Q_NMOS_GDS, Q2 2N7002, Q3 2N7002, Q4 2N7002, T1 TERMINAL_ELEMENT14_5MM_X3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

Commit message: Got oled working.
Parts:
- Q1: value Q_NMOS_GDS -> NVD6828NLT4G; footprint TO_SOT_Packages_THT:TO-220-3_Horizontal -> TO_SOT_Packages_SMD:TO-252-2
- R2, R3, R4, R5: value R -> 100K
- U1: value LM2936-3.3 -> UA78M33CDCY
- U2: footprint Housings_QFP:LQFP-32_7x7mm_Pitch0.8mm -> custom_microcontroller:LQFP-32_7x7mm_Pitch0.8mm
- moved Q1 4.58 mm to (151.2, 90.5), turned to 270 degrees
Routing:
- net Net-(Q1-Pad2): track 13.2 -> 29.8 mm, vias 0 -> 1
- net GND: track 32.5 -> 27.3 mm
